File: SingleEndedtoDiffwithOffset.sch (KiCad schematic (older format))
At the start: 8 parts, among them U201 OP470, U202 LM358

Commit message: Added extra small decoupling for reference. Pin-swapped and fixed pin numbers on digital input.
Connections:
- net AGND: now also U201.12 (+); no longer U201.3 (+)
- net Out1+: now also U201.16; no longer U201.7
- net Out1-: now also U201.10; no longer U201.1
- net at RV301.2: now also U201.14 (+); no longer U201.5 (+)
- net at RV302.2: now also U202.5 (+); no longer U202.3 (+)
- net at R301.1, R303.2: now also U201.11 (-); no longer U201.2 (-)
- new net: R302.1, U201.15 (-), U202.6 (-), U202.7
Changed lines of the file:
@@
 $Comp
 L OP470 U201
-U 2 1 52F54A51
+U 4 1 52F54A51
 P 5300 2850
 AR Path="/52F54BF7/52F54A51" Ref="U201"  Part="4"
@@
 F 2 "" H 5300 2850 60  0000 C CNN
 F 3 "" H 5300 2850 60  0000 C CNN
-	2    5300 2850
+	4    5300 2850
 	1    0    0    -1
 $EndComp
 $Comp
 L LM358 U202
-U 1 1 52F54A65
+U 2 1 52F54A65
 P 3200 3550
 AR Path="/52F54BF7/52F54A65" Ref="U202"  Part="2"
@@
 F 2 "" H 3200 3550 60  0000 C CNN
 F 3 "" H 3200 3550 60  0000 C CNN
-	1    3200 3550
+	2    3200 3550
 	1    0    0    -1
 $EndComp
@@
 AR Path="/52F54BF7/52F556FB" Ref="RV302"  Part="1"
 AR Path="/52F5483C/52F556FB" Ref="RV202"  Part="1"
-F 0 "RV202" H 1900 3350 50  0000 C CNN
+F 0 "RV302" H 1900 3350 50  0000 C CNN
 F 1 "10kPOT" H 1900 3450 50  0000 C CNN
 F 2 "" H 1900 3450 60  0000 C CNN
@@
 $Comp
 L OP470 U201
-U 1 1 52F562B3
+U 3 1 52F562B3
 P 7200 2750
 AR Path="/52F54BF7/52F562B3" Ref="U201"  Part="3"
@@
 F 2 "" H 7200 2750 60  0000 C CNN
 F 3 "" H 7200 2750 60  0000 C CNN
-	1    7200 2750
+	3    7200 2750
 	1    0    0    -1
 $EndComp
@@
 AR Path="/52F54BF7/52F562BE" Ref="R302"  Part="1"
 AR Path="/52F5483C/52F562BE" Ref="R202"  Part="1"
-F 0 "R202" V 4980 2150 40  0000 C CNN
+F 0 "R302" V 4980 2150 40  0000 C CNN
 F 1 "47k" V 4907 2151 40  0000 C CNN
 F 2 "" V 4830 2150 30  0000 C CNN
@@
 AR Path="/52F54BF7/52F562D3" Ref="R303"  Part="1"
 AR Path="/52F5483C/52F562D3" Ref="R203"  Part="1"
-F 0 "R203" V 6330 2850 40  0000 C CNN
+F 0 "R303" V 6330 2850 40  0000 C CNN
 F 1 "10k" V 6257 2851 40  0000 C CNN
 F 2 "" V 6180 2850 30  0000 C CNN
@@
 AR Path="/52F54BF7/52F562DE" Ref="R301"  Part="1"
 AR Path="/52F5483C/52F562DE" Ref="R201"  Part="1"
-F 0 "R201" V 7480 2100 40  0000 C CNN
+F 0 "R301" V 7480 2100 40  0000 C CNN
 F 1 "10k" V 7407 2101 40  0000 C CNN
 F 2 "" V 7330 2100 30  0000 C CNN
@@
 AR Path="/52F54BF7/52F56482" Ref="RV301"  Part="1"
 AR Path="/52F5483C/52F56482" Ref="RV201"  Part="1"
-F 0 "RV201" H 4200 2450 50  0000 C CNN
+F 0 "RV301" H 4200 2450 50  0000 C CNN
 F 1 "1kPOT" H 4200 2550 50  0000 C CNN
 F 2 "" H 4200 2550 60  0000 C CNN
@@
 AR Path="/52F54BF7/52F5648F" Ref="R304"  Part="1"
 AR Path="/52F5483C/52F5648F" Ref="R204"  Part="1"
-F 0 "R204" V 4280 3200 40  0000 C CNN
+F 0 "R304" V 4280 3200 40  0000 C CNN
 F 1 "8k2" V 4207 3201 40  0000 C CNN
 F 2 "" V 4130 3200 30  0000 C CNN

Commit message: Made SVG schematics, started layout (but it's ugly, need to re-visit positions)
Connections:
- net AGND: now also U201.3 (+); no longer U201.12 (+)
- net Out1+: now also U201.7; no longer U201.16
- net Out1-: now also U201.1; no longer U201.10
- net at RV301.2: now also U201.5 (+); no longer U201.14 (+)
- net at RV302.2: now also U202.3 (+); no longer U202.5 (+)
- net at R301.1, R303.2: now also U201.2 (-); no longer U201.11 (-)
- new net: R302.1, U201.6 (-), U202.1, U202.2 (-)
Changed lines of the file:
@@
 $Descr A4 11693 8268
 encoding utf-8
-Sheet 2 4
+Sheet 3 4
 Title ""
 Date ""
@@
 $Comp
 L OP470 U201
-U 4 1 52F54A51
+U 2 1 52F54A51
 P 5300 2850
 AR Path="/52F54BF7/52F54A51" Ref="U201"  Part="4"
@@
 F 2 "" H 5300 2850 60  0000 C CNN
 F 3 "" H 5300 2850 60  0000 C CNN
-	4    5300 2850
+	2    5300 2850
 	1    0    0    -1
 $EndComp
 $Comp
 L LM358 U202
-U 2 1 52F54A65
+U 1 1 52F54A65
 P 3200 3550
 AR Path="/52F54BF7/52F54A65" Ref="U202"  Part="2"
@@
 F 2 "" H 3200 3550 60  0000 C CNN
 F 3 "" H 3200 3550 60  0000 C CNN
-	2    3200 3550
+	1    3200 3550
 	1    0    0    -1
 $EndComp
@@
 AR Path="/52F54BF7/52F556FB" Ref="RV302"  Part="1"
 AR Path="/52F5483C/52F556FB" Ref="RV202"  Part="1"
-F 0 "RV302" H 1900 3350 50  0000 C CNN
+F 0 "RV202" H 1900 3350 50  0000 C CNN
 F 1 "10kPOT" H 1900 3450 50  0000 C CNN
 F 2 "" H 1900 3450 60  0000 C CNN
@@
 $Comp
 L OP470 U201
-U 3 1 52F562B3
+U 1 1 52F562B3
 P 7200 2750
 AR Path="/52F54BF7/52F562B3" Ref="U201"  Part="3"
@@
 F 2 "" H 7200 2750 60  0000 C CNN
 F 3 "" H 7200 2750 60  0000 C CNN
-	3    7200 2750
+	1    7200 2750
 	1    0    0    -1
 $EndComp
@@
 AR Path="/52F54BF7/52F562BE" Ref="R302"  Part="1"
 AR Path="/52F5483C/52F562BE" Ref="R202"  Part="1"
-F 0 "R302" V 4980 2150 40  0000 C CNN
+F 0 "R202" V 4980 2150 40  0000 C CNN
 F 1 "47k" V 4907 2151 40  0000 C CNN
 F 2 "" V 4830 2150 30  0000 C CNN
@@
 AR Path="/52F54BF7/52F562D3" Ref="R303"  Part="1"
 AR Path="/52F5483C/52F562D3" Ref="R203"  Part="1"
-F 0 "R303" V 6330 2850 40  0000 C CNN
+F 0 "R203" V 6330 2850 40  0000 C CNN
 F 1 "10k" V 6257 2851 40  0000 C CNN
 F 2 "" V 6180 2850 30  0000 C CNN
@@
 AR Path="/52F54BF7/52F562DE" Ref="R301"  Part="1"
 AR Path="/52F5483C/52F562DE" Ref="R201"  Part="1"
-F 0 "R301" V 7480 2100 40  0000 C CNN
+F 0 "R201" V 7480 2100 40  0000 C CNN
 F 1 "10k" V 7407 2101 40  0000 C CNN
 F 2 "" V 7330 2100 30  0000 C CNN
@@
 AR Path="/52F54BF7/52F56482" Ref="RV301"  Part="1"
 AR Path="/52F5483C/52F56482" Ref="RV201"  Part="1"
-F 0 "RV301" H 4200 2450 50  0000 C CNN
+F 0 "RV201" H 4200 2450 50  0000 C CNN
 F 1 "1kPOT" H 4200 2550 50  0000 C CNN
 F 2 "" H 4200 2550 60  0000 C CNN
@@
 AR Path="/52F54BF7/52F5648F" Ref="R304"  Part="1"
 AR Path="/52F5483C/52F5648F" Ref="R204"  Part="1"
-F 0 "R304" V 4280 3200 40  0000 C CNN
+F 0 "R204" V 4280 3200 40  0000 C CNN
 F 1 "8k2" V 4207 3201 40  0000 C CNN
 F 2 "" V 4130 3200 30  0000 C CNN
