File: SingleEndedtoDiffwithOffset.sch (KiCad schematic (older format))
At the start: 8 parts, among them U201 OP470, U202 LM358

Commit message: Richard: add 10K pot between LM358 and OP470
Parts:
- added R205: 10k, ~, symbol R
Connections:
- net at R302.1, U201.15 (-): now also R205.1; no longer U202.6 (-), U202.7
- new net: R205.2, U202.6 (-), U202.7
Changed lines of the file:
@@
 LIBS:op470
 LIBS:laser-dac-diff-driver-cache
-EELAYER 24 0
+EELAYER 27 0
 EELAYER END
 $Descr A4 11693 8268
@@
 Sheet 3 4
 Title ""
-Date ""
+Date "5 mar 2014"
 Rev ""
 Comp ""
@@
 	4650 2150 4600 2150
 Wire Wire Line
-	4600 2150 4600 3550
-Wire Wire Line
 	4600 2950 4800 2950
 Connection ~ 3900 3550
@@
 Wire Wire Line
 	5900 3650 8300 3650
+$Comp
+L R R205
+U 1 1 53170122
+P 4600 3300
+AR Path="/52F5483C/53170122" Ref="R205"  Part="1"
+AR Path="/52F54BF7/53170122" Ref="R305"  Part="1"
+F 0 "R305" V 4680 3300 40  0000 C CNN
+F 1 "10k" V 4607 3301 40  0000 C CNN
+F 2 "~" V 4530 3300 30  0000 C CNN
+F 3 "~" H 4600 3300 30  0000 C CNN
+	1    4600 3300
+	1    0    0    -1
+$EndComp
+Wire Wire Line
+	4600 2150 4600 3050
 $EndSCHEMATC

Commit message: SENT TO FAB - also added LC filter to power from 5V to dac, copper pours for Reg heatsinks and missing resistors
Other:
- moved on the sheet: R305
Changed lines of the file:
@@
 EESchema Schematic File Version 2
+LIBS:LM317_HS
 LIBS:74hct04
 LIBS:power
@@
 LIBS:op470
 LIBS:laser-dac-diff-driver-cache
-EELAYER 27 0
+EELAYER 24 0
 EELAYER END
 $Descr A4 11693 8268
 encoding utf-8
-Sheet 3 4
+Sheet 2 4
 Title ""
 Date "5 mar 2014"
@@
 L R R205
 U 1 1 53170122
-P 4600 3300
+P 4600 3250
 AR Path="/52F5483C/53170122" Ref="R205"  Part="1"
 AR Path="/52F54BF7/53170122" Ref="R305"  Part="1"
-F 0 "R305" V 4680 3300 40  0000 C CNN
-F 1 "10k" V 4607 3301 40  0000 C CNN
-F 2 "~" V 4530 3300 30  0000 C CNN
-F 3 "~" H 4600 3300 30  0000 C CNN
-	1    4600 3300
-	1    0    0    -1
-$EndComp
-Wire Wire Line
-	4600 2150 4600 3050
+F 0 "R305" V 4680 3250 40  0000 C CNN
+F 1 "10k" V 4607 3251 40  0000 C CNN
+F 2 "~" V 4530 3250 30  0000 C CNN
+F 3 "~" H 4600 3250 30  0000 C CNN
+	1    4600 3250
+	1    0    0    -1
+$EndComp
+Wire Wire Line
+	4600 3550 4600 3500
+Wire Wire Line
+	4600 2150 4600 3000
 $EndSCHEMATC
