File: laser-dac-diff-driver.kicad_pcb (KiCad board)
At the start: 2 copper layers, 70.5 x 51.4 mm, 55 parts, among them IC401 DCDC-CONV_TRACO_TMH-XXXX_Dual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, P101 CONN_2, P102 CONN_3X2, P103 CONN_6X2, U101 AD5689RARUZ, U102 74HC04, U201 OP470, U202 LM358, U401 LM317EMP, U402 LM317EMP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

Commit message: SENT TO FAB - also added LC filter to power from 5V to dac, copper pours for Reg heatsinks and missing resistors
Parts:
- added C415: 100n, SMD_Packages:SM0603_Capa, F.Cu at (253.0, 82.3)
- added L401: INDUCTOR, SMD_Packages:SM1210, F.Cu at (247.4, 81.5)
- added R205: 10k, Resistors_SMD:Resistor_SMD0805_HandSoldering, F.Cu at (223.3, 49.3)
- added R305: 10k, Resistors_SMD:Resistor_SMD0805_HandSoldering, F.Cu at (223.3, 52.3)
- moved R304 3.32 mm to (223.3, 55.4)
- moved RV301 2.29 mm to (223.5, 62.0)
- moved R204 2.07 mm to (223.3, 46.2)
- moved RV201 1.02 mm to (223.0, 39.6)
Connections:
- net DGND renamed AGND
- R401 pad 1: +5VD -> Net-(L401-Pad2)
- U202 pad 1: Net-(R202-Pad1) -> Net-(R205-Pad2)
- U202 pad 2: Net-(R202-Pad1) -> Net-(R205-Pad2)
- U202 pad 6: Net-(R302-Pad1) -> Net-(R305-Pad2)
- U202 pad 7: Net-(R302-Pad1) -> Net-(R305-Pad2)
- U401 pad 2: +5VD -> Net-(L401-Pad2)
- U401 pad 4: (no net) -> Net-(L401-Pad2)
- U402 pad 4: (no net) -> VAA
- U403 pad 4: (no net) -> /powersupply/-Vout_unreg
Routing:
- net Net-(R202-Pad1): track 53.8 -> 16.6 mm
- net Net-(R205-Pad2): track 0.00 -> 19.1 mm, vias 0 -> 2
- net Net-(L401-Pad2): track 0.00 -> 18.3 mm
- net Net-(R305-Pad2): track 0.00 -> 12.4 mm, vias 0 -> 2
- net +5VD: track 96.1 -> 87.1 mm
- net AGND: track 67.8 -> 75.9 mm, vias 17 -> 16
- net -VAA: track 64.4 -> 59.0 mm
- net Net-(C404-Pad1): track 15.0 -> 18.9 mm
- net Net-(R302-Pad1): track 25.3 -> 28.7 mm, vias 2 -> 0
- net VAA: track 71.8 -> 74.3 mm
- net /MOD_IN: track 94.4 -> 96.5 mm
- net Net-(RV201-Pad2): track 16.0 -> 17.5 mm
- net Net-(R304-Pad2): track 5.88 -> 4.71 mm
- net Net-(R204-Pad2): track 5.62 -> 4.50 mm
- net Net-(RV301-Pad2): track 13.2 -> 14.3 mm, vias 1 -> 0
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- added copper zone on F.Cu, net /powersupply/-Vout_unreg
- added copper zone on F.Cu, net AGND
- added copper zone on F.Cu, net Net-(L401-Pad2)
- added copper zone on F.Cu, net VAA
Other:
- board text added: "FRONT"
- board text added: "github/robot-army /laser-dac-diff-driver BACK"

Commit message: Added bill of materials (shouldn't REALLY be any non-bom changes??)
Parts:
- C101: value C -> 100n
- C102: value C -> 1u; footprint Capacitors_SMD:c_1206 -> SMD_Packages:SM1206
- C103: value C -> 100n; footprint Capacitors_SMD:c_0603 -> SMD_Packages:SM0603_Capa
Routing:
- net +5VD: track 87.1 -> 94.4 mm, vias 0 -> 1
- net AGND: track 75.9 -> 68.5 mm, vias 16 -> 15
